Commit message: workstation: ur5e+ft300+robotiq85+workbench

File: universal_robot/ur_e_description/urdf/ur5e_robot.urdf.xacro (robot description, xacro)
@@ -8,4 +8,8 @@
   <!-- arm -->
   <xacro:ur5e_robot prefix="" joint_limited="false"/>
+  <!-- ft300 -->
+  <xacro:include filename="$(find robotiq_85_gripper)/robotiq_85_description/urdf/robotiq_85_gripper.urdf.xacro" />
+  <!-- robotiq_85 -->
+  <xacro:include filename="$(find robotiq_ft_sensor)/urdf/robotiq_ft300.urdf.xacro" />
   <link name="world" />
   <joint name="world_joint" type="fixed">
@@ -14,3 +18,14 @@
     <origin xyz="0.0 0.0 0.0" rpy="0.0 0.0 0.0" />
   </joint>
+  <!-- ft300 -->
+  <xacro:robotiq_ft300 parent="tool0" prefix="">
+      <origin xyz="0 0 0 " rpy="0 0 0"/>
+  </xacro:robotiq_ft300>
+  <!-- robotiq_85 -->
+ <xacro:robotiq_85_gripper prefix=""/>
+  <joint name="ft_gripper_joint" type="fixed">
+    <parent link="robotiq_ft_frame_id"/>
+    <child link="robotiq_arg2f_base_link"/>
+    <origin xyz="0 0 0" rpy="0 0 0"/>
+  </joint>
 </robot>

Commit message: Finished ur5e workstation robotiq gripper_85 ft300 without linear track.

File: universal_robot/ur_e_description/urdf/ur5e_robot.urdf.xacro (robot description, xacro)
@@ -7,9 +7,9 @@
   <xacro:include filename="$(find ur_e_description)/urdf/ur5e.urdf.xacro" />
   <!-- arm -->
-  <xacro:ur5e_robot prefix="" joint_limited="false"/>
-  <!-- ft300 -->
-  <xacro:include filename="$(find robotiq_85_gripper)/robotiq_85_description/urdf/robotiq_85_gripper.urdf.xacro" />
+  <xacro:ur5e_robot prefix="" joint_limited="true"/>
+  <!-- ft_300 -->
+  <xacro:include filename="$(find robotiq_ft_sensor)/urdf/robotiq_ft300.urdf.xacro" />
   <!-- robotiq_85 -->
-  <xacro:include filename="$(find robotiq_ft_sensor)/urdf/robotiq_ft300.urdf.xacro" />
+  <xacro:include filename="$(find robotiq_85_description)/urdf/robotiq_85_gripper.urdf.xacro" />
   <link name="world" />
   <joint name="world_joint" type="fixed">
@@ -23,9 +23,6 @@
   </xacro:robotiq_ft300>
   <!-- robotiq_85 -->
- <xacro:robotiq_85_gripper prefix=""/>
-  <joint name="ft_gripper_joint" type="fixed">
-    <parent link="robotiq_ft_frame_id"/>
-    <child link="robotiq_arg2f_base_link"/>
-    <origin xyz="0 0 0" rpy="0 0 0"/>
-  </joint>
+  <xacro:robotiq_85_gripper parent="robotiq_ft_frame_id" prefix="">
+      <origin xyz="0 0 0 " rpy="0 ${-pi/2} 0"/>
+  </xacro:robotiq_85_gripper>
 </robot>
